File: usb_csi.kicad_sch (KiCad schematic)
At the start: 25 parts, among them J1 USB_C_Receptacle, J2 USB_C_Receptacle, U1 STM32F103R8Tx

Commit message: Added a switch
Parts:
- added SW1: SW_Push, symbol Switch:SW_Push
Connections:
- net at BT1.2 (-), D20.1 (K), D21.1 (K)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: now also SW1.2
- net at U1.54 (PD2): now also SW1.1
Other:
- moved on the sheet: BT1, D1, D10, D11, D12, D13, D14, D15, D16, D17, D18, D19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

Commit message: Adding USB programmer interface
Parts:
- added J3: USB Programmer, symbol Connector:USB_C_Receptacle
- added R1, R2: 5.1k, symbol Device:R
- added R3: 10k, symbol Device:R
- added SW2: SW_SPDT, symbol Switch:SW_SPDT
- added SW3: SW_Push, symbol Switch:SW_Push
- J1: value USB_C_Receptacle -> USB_C One
- J2: value USB_C_Receptacle -> USB_C Two
Connections:
- net D-: now reaches J2.B10 (RX1-), U1.44 (PA11)
- net D-: now also J3.A7 (D-), J3.B7 (D-)
- net D+: now reaches J2.B6 (D+), U1.45 (PA12)
- net D+: now also J3.A6 (D+), J3.B6 (D+)
- net BOOT0: now reaches U1.60 (BOOT0)
- net BOOT0: now also SW2.2 (B)
- net NRST: now reaches U1.7 (NRST)
- net NRST: now also R3.2, SW3.1
- new net: J3.A4 (VBUS), J3.A9 (VBUS), J3.B4 (VBUS), J3.B9 (VBUS)
- new net: J3.A5 (CC1), R2.1
- new net: J3.B5 (CC2), R1.1
- new net +3.3VP: R3.1, SW2.1 (A)
- new net GND: J3.A1 (GND), J3.A12 (GND), J3.B1 (GND), J3.B12 (GND), J3.S1 (SHIELD), R1.2, R2.2, SW2.3 (C), SW3.2
- no-connect marks 0 -> 11
Other:
- moved on the sheet: BT1, D1, D10, D11, D12, D13, D14, D15, D16, D17, D18, D19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
